Commit message: refactor: migrate MechaBot packages to ASTRA

File: astra_ws/src/astra_description/urdf/astra_base.xacro (robot description, xacro)
@@ -1,4 +1,4 @@
 <?xml version="1.0" ?>
-<robot name="mechabot" xmlns:xacro="http://www.ros.org/wiki/xacro">
+<robot name="astra" xmlns:xacro="http://www.ros.org/wiki/xacro">
     <link name="base_footprint"/>
     <link name="base_link">
@@ -11,14 +11,14 @@
             <origin xyz="0.0 0.0 -0.0125" rpy="0.0 0.0 0.0"/>
             <geometry>
-                <mesh filename="package://mechabot_description/meshes/mechabot_base_link.stl" scale="0.001 0.001 0.001"/>
-            </geometry>
-            <material name="grey">
-                <color rgba="0.8 0.8 0.8 1.0"/>
-            </material>
-        </visual>
-        <collision>
-            <origin xyz="0.0 0.0 -0.0125" rpy="0.0 0.0 0.0"/>
-            <geometry>
-                <mesh filename="package://mechabot_description/meshes/mechabot_base_link.stl" scale="0.001 0.001 0.001"/>
+                <mesh filename="package://astra_description/meshes/astra_base_link.stl" scale="0.001 0.001 0.001"/>
+            </geometry>
+            <material name="grey">
+                <color rgba="0.8 0.8 0.8 1.0"/>
+            </material>
+        </visual>
+        <collision>
+            <origin xyz="0.0 0.0 -0.0125" rpy="0.0 0.0 0.0"/>
+            <geometry>
+                <mesh filename="package://astra_description/meshes/astra_base_link.stl" scale="0.001 0.001 0.001"/>
             </geometry>
             <material name="grey">
@@ -41,5 +41,5 @@
             <origin xyz="0.0 0.0925 -0.034" rpy="0.0 0.0 0.0"/>
             <geometry>
-                <mesh filename="package://mechabot_description/meshes/mechabot_right_wheel.stl" scale="0.001 0.001 0.001"/>
+                <mesh filename="package://astra_description/meshes/astra_right_wheel.stl" scale="0.001 0.001 0.001"/>
             </geometry>
             <material name="blue">
@@ -51,5 +51,5 @@
             <geometry>
                 <sphere radius="0.034"/>
-                <!-- <mesh filename="package://mechabot_description/meshes/mechabot_right_wheel.stl" scale="0.001 0.001 0.001"/> -->
+                <!-- <mesh filename="package://astra_description/meshes/astra_right_wheel.stl" scale="0.001 0.001 0.001"/> -->
             </geometry>
             <material name="blue">
@@ -73,5 +73,5 @@
             <origin xyz="0.0 -0.0925 -0.034" rpy="0.0 0.0 0.0"/>
             <geometry>
-                <mesh filename="package://mechabot_description/meshes/mechabot_left_wheel.stl" scale="0.001 0.001 0.001"/>
+                <mesh filename="package://astra_description/meshes/astra_left_wheel.stl" scale="0.001 0.001 0.001"/>
             </geometry>
             <material name="blue">
@@ -83,5 +83,5 @@
             <geometry>
                 <sphere radius="0.034"/>
-                <!-- <mesh filename="package://mechabot_description/meshes/mechabot_left_wheel.stl" scale="0.001 0.001 0.001"/> -->
+                <!-- <mesh filename="package://astra_description/meshes/astra_left_wheel.stl" scale="0.001 0.001 0.001"/> -->
             </geometry>
             <material name="blue">
@@ -105,15 +105,15 @@
             <origin xyz="-0.085 0.065 -0.021" rpy="0.0 0.0 0.0"/>
             <geometry>
-                <mesh filename="package://mechabot_description/meshes/front_right_castor.stl" scale="0.001 0.001 0.001"/>
-            </geometry>
-            <material name="grey">
-                <color rgba="0.8 0.8 0.8 1.0"/>
-            </material>
-        </visual>
-        <collision>
-            <origin xyz="0.0 0.0 -0.0125" rpy="0.0 0.0 0.0"/>
-            <geometry>
-                <sphere radius="0.00625"/>
-                <!-- <mesh filename="package://mechabot_description/meshes/front_right_castor.stl" scale="0.001 0.001 0.001"/> -->
+                <mesh filename="package://astra_description/meshes/front_right_castor.stl" scale="0.001 0.001 0.001"/>
+            </geometry>
+            <material name="grey">
+                <color rgba="0.8 0.8 0.8 1.0"/>
+            </material>
+        </visual>
+        <collision>
+            <origin xyz="0.0 0.0 -0.0125" rpy="0.0 0.0 0.0"/>
+            <geometry>
+                <sphere radius="0.00625"/>
+                <!-- <mesh filename="package://astra_description/meshes/front_right_castor.stl" scale="0.001 0.001 0.001"/> -->
             </geometry>
             <material name="grey">
@@ -136,15 +136,15 @@
             <origin xyz="-0.085 -0.065 -0.021" rpy="0.0 0.0 0.0"/>
             <geometry>
-                <mesh filename="package://mechabot_description/meshes/front_left_castor.stl" scale="0.001 0.001 0.001"/>
-            </geometry>
-            <material name="grey">
-                <color rgba="0.8 0.8 0.8 1.0"/>
-            </material>
-        </visual>
-        <collision>
-            <origin xyz="0.0 0.0 -0.0125" rpy="0.0 0.0 0.0"/>
-            <geometry>
-                <sphere radius="0.00625"/>
-                <!-- <mesh filename="package://mechabot_description/meshes/front_left_castor.stl" scale="0.001 0.001 0.001"/> -->
+                <mesh filename="package://astra_description/meshes/front_left_castor.stl" scale="0.001 0.001 0.001"/>
+            </geometry>
+            <material name="grey">
+                <color rgba="0.8 0.8 0.8 1.0"/>
+            </material>
+        </visual>
+        <collision>
+            <origin xyz="0.0 0.0 -0.0125" rpy="0.0 0.0 0.0"/>
+            <geometry>
+                <sphere radius="0.00625"/>
+                <!-- <mesh filename="package://astra_description/meshes/front_left_castor.stl" scale="0.001 0.001 0.001"/> -->
             </geometry>
             <material name="grey">
@@ -167,15 +167,15 @@
             <origin xyz="0.085 0.065 -0.0205" rpy="0.0 0.0 0.0"/>
             <geometry>
-                <mesh filename="package://mechabot_description/meshes/rear_right_castor.stl" scale="0.001 0.001 0.001"/>
-            </geometry>
-            <material name="grey">
-                <color rgba="0.8 0.8 0.8 1.0"/>
-            </material>
-        </visual>
-        <collision>
-            <origin xyz="0.0 0.0 -0.0125" rpy="0.0 0.0 0.0"/>
-            <geometry>
-                <sphere radius="0.00625"/>
-                <!-- <mesh filename="package://mechabot_description/meshes/rear_right_castor.stl" scale="0.001 0.001 0.001"/> -->
+                <mesh filename="package://astra_description/meshes/rear_right_castor.stl" scale="0.001 0.001 0.001"/>
+            </geometry>
+            <material name="grey">
+                <color rgba="0.8 0.8 0.8 1.0"/>
+            </material>
+        </visual>
+        <collision>
+            <origin xyz="0.0 0.0 -0.0125" rpy="0.0 0.0 0.0"/>
+            <geometry>
+                <sphere radius="0.00625"/>
+                <!-- <mesh filename="package://astra_description/meshes/rear_right_castor.stl" scale="0.001 0.001 0.001"/> -->
             </geometry>
             <material name="grey">
@@ -198,15 +198,15 @@
             <origin xyz="0.085 -0.065 -0.0205" rpy="0.0 0.0 0.0"/>
             <geometry>
-                <mesh filename="package://mechabot_description/meshes/rear_left_castor.stl" scale="0.001 0.001 0.001"/>
-            </geometry>
-            <material name="grey">
-                <color rgba="0.8 0.8 0.8 1.0"/>
-            </material>
-        </visual>
-        <collision>
-            <origin xyz="0.0 0.0 -0.0125" rpy="0.0 0.0 0.0"/>
-            <geometry>
-                <sphere radius="0.00625"/>
-                <!-- <mesh filename="package://mechabot_description/meshes/rear_left_castor.stl" scale="0.001 0.001 0.001"/> -->
+                <mesh filename="package://astra_description/meshes/rear_left_castor.stl" scale="0.001 0.001 0.001"/>
+            </geometry>
+            <material name="grey">
+                <color rgba="0.8 0.8 0.8 1.0"/>
+            </material>
+        </visual>
+        <collision>
+            <origin xyz="0.0 0.0 -0.0125" rpy="0.0 0.0 0.0"/>
+            <geometry>
+                <sphere radius="0.00625"/>
+                <!-- <mesh filename="package://astra_description/meshes/rear_left_castor.stl" scale="0.001 0.001 0.001"/> -->
             </geometry>
             <material name="grey">
@@ -229,5 +229,5 @@
             <origin xyz="0.0 0.0 -0.1125" rpy="0.0 0.0 0.0"/>
             <geometry>
-                <mesh filename="package://mechabot_description/meshes/mechabot_toplid.stl" scale="0.001 0.001 0.001"/>
+                <mesh filename="package://astra_description/meshes/astra_toplid.stl" scale="0.001 0.001 0.001"/>
             </geometry>
             <material name="red">
@@ -238,5 +238,5 @@
             <origin xyz="0.0 0.0 -0.1125" rpy="0.0 0.0 0.0"/>
             <geometry>
-                <mesh filename="package://mechabot_description/meshes/mechabot_toplid.stl" scale="0.001 0.001 0.001"/>
+                <mesh filename="package://astra_description/meshes/astra_toplid.stl" scale="0.001 0.001 0.001"/>
             </geometry>
             <material name="red">

File: astra_ws/src/astra_description/urdf/astra_gazebo.xacro (robot description, xacro)
@@ -1,4 +1,4 @@
 <?xml version="1.0" ?>
-<robot name="mechabot" xmlns:xacro="http://www.ros.org/wiki/xacro">
+<robot name="astra" xmlns:xacro="http://www.ros.org/wiki/xacro">
     <!-- Wheels -->
     <gazebo reference="right_wheel_link">
@@ -57,5 +57,5 @@
         <!-- ign ros2_control -->
         <plugin filename="ign_ros2_control-system" name="ign_ros2_control::IgnitionROS2ControlPlugin">
-            <parameters>$(find mechabot_controller)/config/mechabot_controllers.yaml</parameters>
+            <parameters>$(find astra_controller)/config/astra_controllers.yaml</parameters>
         </plugin>
         <!-- lidar and camera -->
@@ -66,5 +66,5 @@
         <plugin filename="ignition-gazebo-imu-system" name="ignition::gazebo::systems::Imu"/>
     </gazebo>
-    <!-- MechaBot Sensors-->
+    <!-- astra Sensors-->
     <!-- Lidar -->
     <gazebo reference="lidar_link">

File: astra_ws/src/astra_description/urdf/astra_ros2control.xacro (robot description, xacro)
@@ -1,4 +1,4 @@
 <?xml version="1.0"?>
-<robot name="mechabot" xmlns:xacro="http://www.ros.org/wiki/xacro">
+<robot name="astra" xmlns:xacro="http://www.ros.org/wiki/xacro">
     <ros2_control name="RobotSystem" type="system">
         <!-- ros2_control Gazebo -->
@@ -11,5 +11,5 @@
         <xacro:unless value="$(arg is_sim)">
             <hardware>
-                <plugin>mechabot_firmware/MechabotInterface</plugin>
+                <plugin>astra__firmware/Astra_Interface</plugin>
                 <param name="port">/dev/ttyUSB1</param>
             </hardware>

File: astra_ws/src/astra_description/urdf/astra_sensors.xacro (robot description, xacro)
@@ -1,4 +1,4 @@
 <?xml version="1.0" ?>
-<robot name="mechabot" xmlns:xacro="http://www.ros.org/wiki/xacro">
+<robot name="astra" xmlns:xacro="http://www.ros.org/wiki/xacro">
     <link name="lidar_link">
         <inertial>
@@ -10,5 +10,5 @@
             <origin xyz="-0.028 0.0 -0.132" rpy="0.0 0.0 0.0"/>
             <geometry>
-                <mesh filename="package://mechabot_description/meshes/mechabot_lidar.stl" scale="0.001 0.001 0.001"/>
+                <mesh filename="package://astra_description/meshes/astra_lidar.stl" scale="0.001 0.001 0.001"/>
             </geometry>
             <material name="yellow">
@@ -19,5 +19,5 @@
             <origin xyz="-0.028 0.0 -0.132" rpy="0.0 0.0 0.0"/>
             <geometry>
-                <mesh filename="package://mechabot_description/meshes/mechabot_lidar.stl" scale="0.001 0.001 0.001"/>
+                <mesh filename="package://astra_description/meshes/astra_lidar.stl" scale="0.001 0.001 0.001"/>
             </geometry>
             <material name="yellow">
@@ -40,5 +40,5 @@
             <origin xyz="-0.118 0.0 -0.092" rpy="0.0 0.0 0.0"/>
             <geometry>
-                <mesh filename="package://mechabot_description/meshes/mechabot_camera.stl" scale="0.001 0.001 0.001"/>
+                <mesh filename="package://astra_description/meshes/astra_camera.stl" scale="0.001 0.001 0.001"/>
             </geometry>
             <material name="green">
@@ -49,5 +49,5 @@
             <origin xyz="-0.118 0.0 -0.092" rpy="0.0 0.0 0.0"/>
             <geometry>
-                <mesh filename="package://mechabot_description/meshes/mechabot_camera.stl" scale="0.001 0.001 0.001"/>
+                <mesh filename="package://astra_description/meshes/astra_camera.stl" scale="0.001 0.001 0.001"/>
             </geometry>
             <material name="green">
@@ -76,5 +76,5 @@
             <origin xyz="0.0 0.0 -0.035" rpy="0.0 0.0 0.0"/>
             <geometry>
-                <mesh filename="package://mechabot_description/meshes/mechabot_imu.stl" scale="0.001 0.001 0.001"/>
+                <mesh filename="package://astra_description/meshes/astra_imu.stl" scale="0.001 0.001 0.001"/>
             </geometry>
             <material name="blue">
@@ -85,5 +85,5 @@
             <origin xyz="0.0 0.0 -0.035" rpy="0.0 0.0 0.0"/>
             <geometry>
-                <mesh filename="package://mechabot_description/meshes/mechabot_imu.stl" scale="0.001 0.001 0.001"/>
+                <mesh filename="package://astra_description/meshes/astra_imu.stl" scale="0.001 0.001 0.001"/>
             </geometry>
             <material name="blue">
